Commit message: calibration fizes

File: koko_manufacturing/koko_description_base/robots/koko_description_base.urdf (robot description, URDF)
Before this commit: robot koko_description_base, 2 links, 1 joints
Joints:
- joint base_roll_joint: limit lower=-2.3412 upper=3.3999 effort=0 velocity=0 -> lower=-3.1415 upper=3.1415 effort=0 velocity=0

File: koko_manufacturing/koko_description_link/robots/koko_description_link.urdf (robot description, URDF)
Before this commit: robot koko_description_link, 3 links, 2 joints
Joints:
- joint lift_joint: limit lower=-2.2944 upper=1.0 effort=0 velocity=0 -> lower=-3.141592 upper=3.141592 effort=0 velocity=0
- joint roll_joint: limit lower=-2.6761 upper=2.6761 effort=0 velocity=0 -> lower=-3.141592 upper=3.141592 effort=0 velocity=0
