Commit message: improved pose target converter with posture control

File: koko_gazebo/robots/koko_description_sevendof_kin.urdf (robot description, URDF)
Before this commit: robot koko_description_sevendof_kin, 14 links, 13 joints
Links:
- removed link kinect_link
Joints:
- removed joint kinect_joint
