Commit message: working dexnet

File: blue_dexnet/urdf/primesense_v0/primesense.urdf.xacro (robot description, xacro)
@@ -59,5 +59,5 @@
     </joint>
     <link
-      name="primesense_link">
+      name="camera_link">
       <inertial>
         <origin
@@ -101,11 +101,15 @@
       name="primesense_joint"
       type="fixed">
+      <!-- Pre-Brent's edits -->
+      <!-- <origin -->
+        <!-- xyz="0.011494 0.33383 0.61099" -->
+        <!-- rpy="-1.5708 1.5708 -3.1416" /> -->
       <origin
-        xyz="0.011494 0.33383 0.61099"
-        rpy="3.1416 2.609E-15 -3.1416" />
+        xyz="0.116494 0.33383 0.72599"
+        rpy="-1.5708 1.5708 -3.1416" />
       <parent
         link="camera_base_link" />
       <child
-        link="primesense_link" />
+        link="camera_link" />
       <axis
         xyz="0 0 0" />

Commit message: running! but need to debug

File: blue_dexnet/urdf/primesense_v0/primesense.urdf.xacro (robot description, xacro)
@@ -59,5 +59,5 @@
     </joint>
     <link
-      name="camera_link">
+      name="camera_depth_optical_frame">
       <inertial>
         <origin
@@ -102,14 +102,15 @@
       type="fixed">
       <!-- Pre-Brent's edits -->
+      <origin
+        xyz="0.014494 0.33383 0.71099"
+        rpy="3.1416 2.609E-15 -3.1416" />
+      <!-- rpy="-1.5708 1.5708 -3.1416" /> -->
       <!-- <origin -->
-        <!-- xyz="0.011494 0.33383 0.61099" -->
+        <!-- xyz="0.116494 0.33383 0.72599" -->
         <!-- rpy="-1.5708 1.5708 -3.1416" /> -->
-      <origin
-        xyz="0.116494 0.33383 0.72599"
-        rpy="-1.5708 1.5708 -3.1416" />
       <parent
         link="camera_base_link" />
       <child
-        link="camera_link" />
+        link="camera_depth_optical_frame" />
       <axis
         xyz="0 0 0" />
